File: for-science.sch (KiCad schematic (older format))
At the start: 53 parts, among them J1 TRRS, J2 TRRS, U1 ARDUINO_PRO_MICRO

Commit message: Update SCH from KiCad v2 to v5
Parts:
- D1, D10, D11, D13, D14, D15, D16, D17, D19, D2, D20, D21, D22, D23, D26, D27, D28, D3, D4, D5, D7, D8, D9: symbol DIODE -> for-science-rescue:DIODE
- EXTRADATA1, GROUND1, RESET1, TX0: symbol Conn_01x01 -> for-science-rescue:Conn_01x01
- J1, J2: symbol Audio-Jack-4 -> for-science-rescue:Audio-Jack-4
- MX0:0, MX0:1, MX0:2, MX0:3, MX0:4, MX1:0, MX1:1, MX1:2, MX1:3, MX1:4, MX2:0, MX2:1, MX2:2, MX2:3, MX2:4, MX3:0, MX3:1, MX3:2, MX3:3, MX3:4, MX4:2, MX4:3, MX4:4: symbol SWITCH_PUSH -> for-science-rescue:SWITCH_PUSH
- U1: symbol ARDUINO_PRO_MICRO-RESCUE-for-science -> for-science-rescue:ARDUINO_PRO_MICRO-RESCUE-for-science
Connections:
- wire segments 26 -> 64
